Commit message: First version of new robot_dart

File: res/models/arm.urdf (robot description, URDF)
Before this commit: robot omnipointer, 7 links, 6 joints
Links:
- link arm_link_5: mass None -> 1e-8
Joints:
- joint arm_joint_1: limit lower=-3.1415926535 upper=3.1415926535 effort=30.0 velocity=5.0 -> lower=-3.1415926535 upper=3.1415926535 effort=5.0 velocity=5.0
- joint arm_joint_2: limit lower=-1.57079632679 upper=1.57079632679 effort=30.0 velocity=5.0 -> lower=-1.57079632679 upper=1.57079632679 effort=5.0 velocity=5.0
- joint arm_joint_3: limit lower=-1.57079632679 upper=1.57079632679 effort=30.0 velocity=5.0 -> lower=-1.57079632679 upper=1.57079632679 effort=5.0 velocity=5.0
- joint arm_joint_4: limit lower=-1.57079632679 upper=1.57079632679 effort=30.0 velocity=5.0 -> lower=-1.57079632679 upper=1.57079632679 effort=5.0 velocity=5.0
