Commit message: our Talos has red grippers!

File: robots/talos/talos.urdf (robot description, URDF)
Before this commit: robot talos, 60 links, 59 joints
Links:
- link arm_left_1_link: geometry collision mesh filename=package://talos_description/meshes/arm/arm_1_collision.glb scale=1 1 1; visual mesh filename=package://talos_description/meshes/arm/arm_1.glb scale=1 1 1
- link arm_left_2_link: geometry collision mesh filename=package://talos_description/meshes/arm/arm_2_collision.glb scale=1 1 1; visual mesh filename=package://talos_description/meshes/arm/arm_2.glb scale=1 1 1
- link arm_left_3_link: geometry collision mesh filename=package://talos_description/meshes/arm/arm_3_collision.glb scale=1 1 1; visual mesh filename=package://talos_description/meshes/arm/arm_3.glb scale=1 1 1
- link arm_left_4_link: geometry collision mesh filename=package://talos_description/meshes/arm/arm_4_collision.glb scale=1 1 1; visual mesh filename=package://talos_description/meshes/arm/arm_4.glb scale=1 1 1
- link arm_left_5_link: geometry collision mesh filename=package://talos_description/meshes/arm/arm_5_collision.glb scale=1 1 1; visual mesh filename=package://talos_description/meshes/arm/arm_5.glb scale=1 1 1
- link arm_left_6_link: geometry collision mesh filename=package://talos_description/meshes/arm/arm_6_collision.glb scale=1 1 1; visual mesh filename=package://talos_description/meshes/arm/arm_6.glb scale=1 1 1
- link arm_left_7_link: geometry collision mesh filename=package://talos_description/meshes/arm/arm_7_collision.glb scale=1 1 1; visual mesh filename=package://talos_description/meshes/arm/arm_7.glb scale=1 1 1
- link arm_right_1_link: geometry collision mesh filename=package://talos_description/meshes/arm/arm_1_collision.glb scale=1 -1 1; visual mesh filename=package://talos_description/meshes/arm/arm_1.glb scale=1 -1 1
- link arm_right_2_link: geometry collision mesh filename=package://talos_description/meshes/arm/arm_2_collision.glb scale=1 -1 1; visual mesh filename=package://talos_description/meshes/arm/arm_2.glb scale=1 -1 1
- link arm_right_3_link: geometry collision mesh filename=package://talos_description/meshes/arm/arm_3_collision.glb scale=1 -1 1; visual mesh filename=package://talos_description/meshes/arm/arm_3.glb scale=1 -1 1
- link arm_right_4_link: geometry collision mesh filename=package://talos_description/meshes/arm/arm_4_collision.glb scale=1 -1 1; visual mesh filename=package://talos_description/meshes/arm/arm_4.glb scale=1 -1 1
- link arm_right_5_link: geometry collision mesh filename=package://talos_description/meshes/arm/arm_5_collision.glb scale=1 -1 1; visual mesh filename=package://talos_description/meshes/arm/arm_5.glb scale=1 -1 1
- link arm_right_6_link: geometry collision mesh filename=package://talos_description/meshes/arm/arm_6_collision.glb scale=1 -1 1; visual mesh filename=package://talos_description/meshes/arm/arm_6.glb scale=1 -1 1
- link arm_right_7_link: geometry collision mesh filename=package://talos_description/meshes/arm/arm_7_collision.glb scale=1 -1 1; visual mesh filename=package://talos_description/meshes/arm/arm_7.glb scale=1 -1 1
- link base_link: geometry collision mesh filename=package://talos_description/meshes/torso/base_link_collisio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 scale=1 1 1; visual mesh filename=package://talos_description/meshes/torso/base_link.glb scale=1 1 1
- link gripper_left_base_link: geometry collision mesh filename=package://talos_description/meshes/gripper/base_link_collis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 scale=1 1 1; visual mesh filename=package://talos_description/meshes/gripper/base_link.glb scale=1 1 1
- link gripper_left_fingertip_1_link: geometry collision mesh filename=package://talos_description/meshes/gripper/fingertip_collis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 scale=1 1 1; visual mesh filename=package://talos_description/meshes/gripper/fingertip.glb scale=1 1 1
- link gripper_left_fingertip_2_link: geometry collision mesh filename=package://talos_description/meshes/gripper/fingertip_collis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 scale=1 1 1; visual mesh filename=package://talos_description/meshes/gripper/fingertip.glb scale=1 1 1
- link gripper_left_fingertip_3_link: geometry collision mesh filename=package://talos_description/meshes/gripper/fingertip_collis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 scale=1 1 1; visual mesh filename=package://talos_description/meshes/gripper/fingertip.glb scale=1 1 1
- link gripper_left_inner_double_link: geometry collision mesh filename=package://talos_description/meshes/gripper/inner_double_col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 scale=1 1 1; visual mesh filename=package://talos_description/meshes/gripper/inner_double.glb scale=1 1 1
- link gripper_left_inner_single_link: geometry collision mesh filename=package://talos_description/meshes/gripper/inner_single_col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 scale=1 1 1; visual mesh filename=package://talos_description/meshes/gripper/inner_single.glb scale=1 1 1
- link gripper_right_base_link: geometry collision mesh filename=package://talos_description/meshes/gripper/base_link_collis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 scale=1 1 1; visual mesh filename=package://talos_description/meshes/gripper/base_link.glb scale=1 1 1
- link gripper_right_fingertip_1_link: geometry collision mesh filename=package://talos_description/meshes/gripper/fingertip_collis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 scale=1 1 1; visual mesh filename=package://talos_description/meshes/gripper/fingertip.glb scale=1 1 1
- link gripper_right_fingertip_2_link: geometry collision mesh filename=package://talos_description/meshes/gripper/fingertip_collis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 scale=1 1 1; visual mesh filename=package://talos_description/meshes/gripper/fingertip.glb scale=1 1 1
- link gripper_right_fingertip_3_link: geometry collision mesh filename=package://talos_description/meshes/gripper/fingertip_collis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 scale=1 1 1; visual mesh filename=package://talos_description/meshes/gripper/fingertip.glb scale=1 1 1
- link gripper_right_inner_double_link: geometry collision mesh filename=package://talos_description/meshes/gripper/inner_double_col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 scale=1 1 1; visual mesh filename=package://talos_description/meshes/gripper/inner_double.glb scale=1 1 1
- link gripper_right_inner_single_link: geometry collision mesh filename=package://talos_description/meshes/gripper/inner_single_col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 scale=1 1 1; visual mesh filename=package://talos_description/meshes/gripper/inner_single.glb scale=1 1 1
- link head_1_link: geometry collision mesh filename=package://talos_description/meshes/head/head_1_collision.glb scale=1 1 1; visual mesh filename=package://talos_description/meshes/head/head_1.glb scale=1 1 1
- link head_2_link: geometry collision mesh filename=package://talos_description/meshes/head/head_2_collision.glb scale=1 1 1; visual mesh filename=package://talos_description/meshes/head/head_2.glb scale=1 1 1
- link leg_left_1_link: geometry collision mesh filename=package://talos_description/meshes/v2/hip_z_collision.glb scale=1 1 1; visual mesh filename=package://talos_description/meshes/v2/hip_z_lo_res.glb scale=1 1 1
- link leg_left_2_link: geometry collision mesh filename=package://talos_description/meshes/v2/hip_x_collision.glb scale=1 1 1; visual mesh filename=package://talos_description/meshes/v2/hip_x_lo_res.glb scale=1 1 1
- link leg_left_3_link: geometry collision mesh filename=package://talos_description/meshes/v2/hip_y_collision.glb scale=1 1 1; visual mesh filename=package://talos_description/meshes/v2/hip_y_lo_res.glb scale=1 1 1
- link leg_left_4_link: geometry collision mesh filename=package://talos_description/meshes/v2/knee_collision.glb scale=1 1 1; visual mesh filename=package://talos_description/meshes/v2/knee_lo_res.glb scale=1 1 1
- link leg_left_5_link: geometry collision mesh filename=package://talos_description/meshes/v2/ankle_Y_collision.glb scale=1 1 1; visual mesh filename=package://talos_description/meshes/v2/ankle_Y_lo_res.glb scale=1 1 1
- link leg_left_6_link: geometry collision mesh filename=package://talos_description/meshes/v2/ankle_X_collision.glb scale=1 1 1; visual mesh filename=package://talos_description/meshes/v2/ankle_X_lo_res.glb scale=1 1 1
- link leg_right_1_link: geometry collision mesh filename=package://talos_description/meshes/v2/hip_z_collision.glb scale=1 -1 1; visual mesh filename=package://talos_description/meshes/v2/hip_z_lo_res.glb scale=1 -1 1
- link leg_right_2_link: geometry collision mesh filename=package://talos_description/meshes/v2/hip_x_collision.glb scale=1 -1 1; visual mesh filename=package://talos_description/meshes/v2/hip_x_lo_res.glb scale=1 -1 1
- link leg_right_3_link: geometry collision mesh filename=package://talos_description/meshes/v2/hip_y_collision.glb scale=1 -1 1; visual mesh filename=package://talos_description/meshes/v2/hip_y_lo_res.glb scale=1 -1 1
- link leg_right_4_link: geometry collision mesh filename=package://talos_description/meshes/v2/knee_collision.glb scale=1 -1 1; visual mesh filename=package://talos_description/meshes/v2/knee_lo_res.glb scale=1 -1 1
- link leg_right_5_link: geometry collision mesh filename=package://talos_description/meshes/v2/ankle_Y_collision.glb scale=1 -1 1; visual mesh filename=package://talos_description/meshes/v2/ankle_Y_lo_res.glb scale=1 -1 1
- link leg_right_6_link: geometry collision mesh filename=package://talos_description/meshes/v2/ankle_X_collision.glb scale=1 -1 1; visual mesh filename=package://talos_description/meshes/v2/ankle_X_lo_res.glb scale=1 -1 1
- link rgbd_link: geometry collision box size=0.04 0.185 0.03; visual mesh filename=package://talos_description/meshes/sensors/orbbec/orbbec.glb
- link torso_1_link: geometry collision mesh filename=package://talos_description/meshes/torso/torso_1.glb scale=1 1 1; visual mesh filename=package://talos_description/meshes/torso/torso_1.glb scale=1 1 1
- link torso_2_link: geometry collision mesh filename=package://talos_description/meshes/torso/torso_2_collision.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 scale=1 1 1; visual mesh filename=package://talos_description/meshes/torso/torso_2.glb scale=1 1 1
