Commit message: [icub]: fix collision meshes

File: robots/icub/icub.urdf (robot description, URDF)
Before this commit: robot icub, 48 links, 47 joints
Links:
- link chest: geometry collision mesh filename=package://icub_description/meshes/collision/obj/icub_simple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; visual mesh filename=package://icub_description/meshes/visual/dae/icub_chest.dae
- link head: geometry collision mesh filename=package://icub_description/meshes/collision/obj/icub_simple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; visual mesh filename=package://icub_description/meshes/visual/dae/icub_head.dae
- link l_ankle_1: geometry collision mesh filename=package://icub_description/meshes/collision/obj/icub_simple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; visual mesh filename=package://icub_description/meshes/visual/dae/icub_l_ankle_1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
- link l_ankle_2: geometry collision mesh filename=package://icub_description/meshes/collision/obj/icub_simple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; visual mesh filename=package://icub_description/meshes/visual/dae/icub_l_ankle_2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
- link l_elbow_1: geometry collision mesh filename=package://icub_description/meshes/collision/obj/icub_simple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; visual mesh filename=package://icub_description/meshes/visual/dae/icub_l_elbow_1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
- link l_forearm: geometry collision mesh filename=package://icub_description/meshes/collision/obj/icub_simple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; visual mesh filename=package://icub_description/meshes/visual/dae/icub_l_forearm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
- link l_hand: geometry collision mesh filename=package://icub_description/meshes/collision/obj/icub_simple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 scale=1 1 1; visual mesh filename=package://icub_description/meshes/visual/dae/icub_l_hand.dae scale=1 1 1
- link l_hip_pitch_link: geometry collision mesh filename=package://icub_description/meshes/collision/obj/icub_simple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; visual mesh filename=package://icub_description/meshes/visual/dae/icub_l_hip_pit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
- link l_hip_roll_link: geometry collision mesh filename=package://icub_description/meshes/collision/obj/icub_simple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; visual mesh filename=package://icub_description/meshes/visual/dae/icub_l_hip_rol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
- link l_hip_yaw_link: geometry collision mesh filename=package://icub_description/meshes/collision/obj/icub_simple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; visual mesh filename=package://icub_description/meshes/visual/dae/icub_l_hip_yaw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
- link l_lower_leg: geometry collision mesh filename=package://icub_description/meshes/collision/obj/icub_simple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; visual mesh filename=package://icub_description/meshes/visual/dae/icub_l_lower_l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
- link l_shoulder_pitch_link: geometry collision mesh filename=package://icub_description/meshes/collision/obj/icub_simple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; visual mesh filename=package://icub_description/meshes/visual/dae/icub_l_shoulde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
- link l_shoulder_roll_link: geometry collision mesh filename=package://icub_description/meshes/collision/obj/icub_simple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; visual mesh filename=package://icub_description/meshes/visual/dae/icub_l_shoulde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
- link l_shoulder_yaw_link: geometry collision mesh filename=package://icub_description/meshes/collision/obj/icub_simple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; visual mesh filename=package://icub_description/meshes/visual/dae/icub_l_shoulde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
- link l_upper_arm: geometry collision mesh filename=package://icub_description/meshes/collision/obj/icub_simple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; visual mesh filename=package://icub_description/meshes/visual/dae/icub_l_upper_a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
- link l_upper_leg: geometry collision mesh filename=package://icub_description/meshes/collision/obj/icub_simple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; visual mesh filename=package://icub_description/meshes/visual/dae/icub_l_upper_l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
- link l_wrist_1: geometry collision mesh filename=package://icub_description/meshes/collision/obj/icub_simple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; visual mesh filename=package://icub_description/meshes/visual/dae/icub_l_wrist_1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
- link lap_belt_1: geometry collision mesh filename=package://icub_description/meshes/collision/obj/icub_simple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; visual mesh filename=package://icub_description/meshes/visual/dae/icub_lap_belt_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
- link lap_belt_2: geometry collision mesh filename=package://icub_description/meshes/collision/obj/icub_simple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; visual mesh filename=package://icub_description/meshes/visual/dae/icub_lap_belt_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
- link neck_roll_link: geometry collision mesh filename=package://icub_description/meshes/collision/obj/icub_simple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; visual mesh filename=package://icub_description/meshes/visual/dae/icub_neck_roll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
- link neck_yaw_link: geometry collision mesh filename=package://icub_description/meshes/collision/obj/icub_simple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; visual mesh filename=package://icub_description/meshes/visual/dae/icub_neck_yaw_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
- link r_ankle_1: geometry collision mesh filename=package://icub_description/meshes/collision/obj/icub_simple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; visual mesh filename=package://icub_description/meshes/visual/dae/icub_r_ankle_1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
- link r_ankle_2: geometry collision mesh filename=package://icub_description/meshes/collision/obj/icub_simple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; visual mesh filename=package://icub_description/meshes/visual/dae/icub_r_ankle_2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
- link r_elbow_1: geometry collision mesh filename=package://icub_description/meshes/collision/obj/icub_simple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; visual mesh filename=package://icub_description/meshes/visual/dae/icub_r_elbow_1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
- link r_forearm: geometry collision mesh filename=package://icub_description/meshes/collision/obj/icub_simple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; visual mesh filename=package://icub_description/meshes/visual/dae/icub_r_forearm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
- link r_hand: geometry collision mesh filename=package://icub_description/meshes/collision/obj/icub_simple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 scale=1 1 1; visual mesh filename=package://icub_description/meshes/visual/dae/icub_r_hand.dae scale=1 1 1
- link r_hip_pitch_link: geometry collision mesh filename=package://icub_description/meshes/collision/obj/icub_simple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; visual mesh filename=package://icub_description/meshes/visual/dae/icub_r_hip_pit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
- link r_hip_roll_link: geometry collision mesh filename=package://icub_description/meshes/collision/obj/icub_simple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; visual mesh filename=package://icub_description/meshes/visual/dae/icub_r_hip_rol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
- link r_hip_yaw_link: geometry collision mesh filename=package://icub_description/meshes/collision/obj/icub_simple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; visual mesh filename=package://icub_description/meshes/visual/dae/icub_r_hip_yaw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
- link r_lower_leg: geometry collision mesh filename=package://icub_description/meshes/collision/obj/icub_simple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; visual mesh filename=package://icub_description/meshes/visual/dae/icub_r_lower_l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
- link r_shoulder_pitch_link: geometry collision mesh filename=package://icub_description/meshes/collision/obj/icub_simple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; visual mesh filename=package://icub_description/meshes/visual/dae/icub_r_shoulde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
- link r_shoulder_roll_link: geometry collision mesh filename=package://icub_description/meshes/collision/obj/icub_simple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; visual mesh filename=package://icub_description/meshes/visual/dae/icub_r_shoulde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
- link r_shoulder_yaw_link: geometry collision mesh filename=package://icub_description/meshes/collision/obj/icub_simple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; visual mesh filename=package://icub_description/meshes/visual/dae/icub_r_shoulde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
- link r_upper_arm: geometry collision mesh filename=package://icub_description/meshes/collision/obj/icub_simple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; visual mesh filename=package://icub_description/meshes/visual/dae/icub_r_upper_a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
- link r_upper_leg: geometry collision mesh filename=package://icub_description/meshes/collision/obj/icub_simple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; visual mesh filename=package://icub_description/meshes/visual/dae/icub_r_upper_l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
- link r_wrist_1: geometry collision mesh filename=package://icub_description/meshes/collision/obj/icub_simple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; visual mesh filename=package://icub_description/meshes/visual/dae/icub_r_wrist_1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
- link waist: geometry collision mesh filename=package://icub_description/meshes/collision/obj/icub_simple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; visual mesh filename=package://icub_description/meshes/visual/dae/icub_waist.dae

Commit message: add glb for iCub

File: robots/icub/icub.urdf (robot description, URDF)
Before this commit: robot icub, 48 links, 47 joints
Links:
- link chest: geometry collision mesh filename=package://icub_description/meshes/collision/obj/icub_simple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; visual mesh filename=package://icub_description/meshes/visual/glb/icub_chest.glb
- link head: geometry collision mesh filename=package://icub_description/meshes/collision/obj/icub_simple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; visual mesh filename=package://icub_description/meshes/visual/glb/icub_head.glb
- link l_ankle_1: geometry collision mesh filename=package://icub_description/meshes/collision/obj/icub_simple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; visual mesh filename=package://icub_description/meshes/visual/glb/icub_l_ankle_1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
- link l_ankle_2: geometry collision mesh filename=package://icub_description/meshes/collision/obj/icub_simple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; visual mesh filename=package://icub_description/meshes/visual/glb/icub_l_ankle_2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
- link l_elbow_1: geometry collision mesh filename=package://icub_description/meshes/collision/obj/icub_simple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; visual mesh filename=package://icub_description/meshes/visual/glb/icub_l_elbow_1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
- link l_forearm: geometry collision mesh filename=package://icub_description/meshes/collision/obj/icub_simple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; visual mesh filename=package://icub_description/meshes/visual/glb/icub_l_forearm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
- link l_hand: geometry collision mesh filename=package://icub_description/meshes/collision/obj/icub_simple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 scale=1 1 1; visual mesh filename=package://icub_description/meshes/visual/glb/icub_l_hand.glb scale=1 1 1
- link l_hip_pitch_link: geometry collision mesh filename=package://icub_description/meshes/collision/obj/icub_simple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; visual mesh filename=package://icub_description/meshes/visual/glb/icub_l_hip_pit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
- link l_hip_roll_link: geometry collision mesh filename=package://icub_description/meshes/collision/obj/icub_simple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; visual mesh filename=package://icub_description/meshes/visual/glb/icub_l_hip_rol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
- link l_hip_yaw_link: geometry collision mesh filename=package://icub_description/meshes/collision/obj/icub_simple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; visual mesh filename=package://icub_description/meshes/visual/glb/icub_l_hip_yaw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
- link l_lower_leg: geometry collision mesh filename=package://icub_description/meshes/collision/obj/icub_simple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; visual mesh filename=package://icub_description/meshes/visual/glb/icub_l_lower_l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
- link l_shoulder_pitch_link: geometry collision mesh filename=package://icub_description/meshes/collision/obj/icub_simple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; visual mesh filename=package://icub_description/meshes/visual/glb/icub_l_shoulde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
- link l_shoulder_roll_link: geometry collision mesh filename=package://icub_description/meshes/collision/obj/icub_simple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; visual mesh filename=package://icub_description/meshes/visual/glb/icub_l_shoulde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
- link l_shoulder_yaw_link: geometry collision mesh filename=package://icub_description/meshes/collision/obj/icub_simple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; visual mesh filename=package://icub_description/meshes/visual/glb/icub_l_shoulde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
- link l_upper_arm: geometry collision mesh filename=package://icub_description/meshes/collision/obj/icub_simple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; visual mesh filename=package://icub_description/meshes/visual/glb/icub_l_upper_a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
- link l_upper_leg: geometry collision mesh filename=package://icub_description/meshes/collision/obj/icub_simple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; visual mesh filename=package://icub_description/meshes/visual/glb/icub_l_upper_l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
- link l_wrist_1: geometry collision mesh filename=package://icub_description/meshes/collision/obj/icub_simple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; visual mesh filename=package://icub_description/meshes/visual/glb/icub_l_wrist_1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
- link lap_belt_1: geometry collision mesh filename=package://icub_description/meshes/collision/obj/icub_simple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; visual mesh filename=package://icub_description/meshes/visual/glb/icub_lap_belt_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
- link lap_belt_2: geometry collision mesh filename=package://icub_description/meshes/collision/obj/icub_simple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; visual mesh filename=package://icub_description/meshes/visual/glb/icub_lap_belt_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
- link left_foot: geometry collision box size=0.09 0.035 0.2; visual mesh filename=package://icub_description/meshes/visual/glb/icub_l_foot.glb
- link neck_roll_link: geometry collision mesh filename=package://icub_description/meshes/collision/obj/icub_simple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; visual mesh filename=package://icub_description/meshes/visual/glb/icub_neck_roll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
- link neck_yaw_link: geometry collision mesh filename=package://icub_description/meshes/collision/obj/icub_simple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; visual mesh filename=package://icub_description/meshes/visual/glb/icub_neck_yaw_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
- link r_ankle_1: geometry collision mesh filename=package://icub_description/meshes/collision/obj/icub_simple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; visual mesh filename=package://icub_description/meshes/visual/glb/icub_r_ankle_1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
- link r_ankle_2: geometry collision mesh filename=package://icub_description/meshes/collision/obj/icub_simple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; visual mesh filename=package://icub_description/meshes/visual/glb/icub_r_ankle_2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
- link r_elbow_1: geometry collision mesh filename=package://icub_description/meshes/collision/obj/icub_simple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; visual mesh filename=package://icub_description/meshes/visual/glb/icub_r_elbow_1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
- link r_forearm: geometry collision mesh filename=package://icub_description/meshes/collision/obj/icub_simple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; visual mesh filename=package://icub_description/meshes/visual/glb/icub_r_forearm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
- link r_hand: geometry collision mesh filename=package://icub_description/meshes/collision/obj/icub_simple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 scale=1 1 1; visual mesh filename=package://icub_description/meshes/visual/glb/icub_r_hand.glb scale=1 1 1
- link r_hip_pitch_link: geometry collision mesh filename=package://icub_description/meshes/collision/obj/icub_simple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; visual mesh filename=package://icub_description/meshes/visual/glb/icub_r_hip_pit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
- link r_hip_roll_link: geometry collision mesh filename=package://icub_description/meshes/collision/obj/icub_simple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; visual mesh filename=package://icub_description/meshes/visual/glb/icub_r_hip_rol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
- link r_hip_yaw_link: geometry collision mesh filename=package://icub_description/meshes/collision/obj/icub_simple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; visual mesh filename=package://icub_description/meshes/visual/glb/icub_r_hip_yaw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
- link r_lower_leg: geometry collision mesh filename=package://icub_description/meshes/collision/obj/icub_simple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; visual mesh filename=package://icub_description/meshes/visual/glb/icub_r_lower_l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
- link r_shoulder_pitch_link: geometry collision mesh filename=package://icub_description/meshes/collision/obj/icub_simple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; visual mesh filename=package://icub_description/meshes/visual/glb/icub_r_shoulde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
- link r_shoulder_roll_link: geometry collision mesh filename=package://icub_description/meshes/collision/obj/icub_simple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; visual mesh filename=package://icub_description/meshes/visual/glb/icub_r_shoulde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
- link r_shoulder_yaw_link: geometry collision mesh filename=package://icub_description/meshes/collision/obj/icub_simple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; visual mesh filename=package://icub_description/meshes/visual/glb/icub_r_shoulde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
- link r_upper_arm: geometry collision mesh filename=package://icub_description/meshes/collision/obj/icub_simple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; visual mesh filename=package://icub_description/meshes/visual/glb/icub_r_upper_a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
- link r_upper_leg: geometry collision mesh filename=package://icub_description/meshes/collision/obj/icub_simple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; visual mesh filename=package://icub_description/meshes/visual/glb/icub_r_upper_l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
- link r_wrist_1: geometry collision mesh filename=package://icub_description/meshes/collision/obj/icub_simple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; visual mesh filename=package://icub_description/meshes/visual/glb/icub_r_wrist_1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
- link right_foot: geometry collision box size=0.09 0.035 0.2; visual mesh filename=package://icub_description/meshes/visual/glb/icub_r_foot.glb
- link waist: geometry collision mesh filename=package://icub_description/meshes/collision/obj/icub_simple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; visual mesh filename=package://icub_description/meshes/visual/glb/icub_waist.glb
