Commit message: [iiwa]: make it consistent with other robots

File: robots/iiwa/iiwa.urdf (robot description, URDF)
Before this commit: robot iiwa14, 10 links, 9 joints
Links:
- link iiwa_link_0: geometry collision box size=0.24 0.23 0.1575; visual mesh filename=package://iiwa_description/meshes/link_0.stl
- link iiwa_link_1: geometry collision box size=0.175 0.19 0.26; visual mesh filename=package://iiwa_description/meshes/link_1.stl
- link iiwa_link_2: geometry collision box size=0.175 0.24 0.19; visual mesh filename=package://iiwa_description/meshes/link_2.stl
- link iiwa_link_3: geometry collision box size=0.125 0.15 0.26; visual mesh filename=package://iiwa_description/meshes/link_3.stl
- link iiwa_link_4: geometry collision box size=0.125 0.22 0.15; visual mesh filename=package://iiwa_description/meshes/link_4.stl
- link iiwa_link_5: geometry collision box size=0.125 0.15 0.24; visual mesh filename=package://iiwa_description/meshes/link_5.stl
- link iiwa_link_6: geometry collision box size=0.125 0.15 0.125; visual mesh filename=package://iiwa_description/meshes/link_6.stl
- link iiwa_link_7: geometry collision box size=0.1 0.1 0.05; visual mesh filename=package://iiwa_description/meshes/link_7.stl
