Commit message: [robots]: new Franka URDF and minor adaptation of example

File: robots/franka/franka.urdf (robot description, URDF)
Before this commit: robot franka, 11 links, 10 joints
Links:
- removed link box
- removed link world
- added link panda_hand, mass 0.68; collision mesh filename=package://franka_description/meshes/collision/hand.stl; visual mesh filename=package://franka_description/meshes/visual/hand.dae
- added link panda_leftfinger, mass 0.01; collision mesh filename=package://franka_description/meshes/collision/finger.stl; visual mesh filename=package://franka_description/meshes/visual/finger.dae
- added link panda_rightfinger, mass 0.01; collision mesh filename=package://franka_description/meshes/collision/finger.stl; visual mesh filename=package://franka_description/meshes/visual/finger.dae
- link panda_link0: mass 1.2 -> 3.06
- link panda_link1: mass 2.0 -> 2.34; geometry collision mesh filename=package://franka_description/meshes/collision/link1.stl; visual mesh filename=package://franka_description/meshes/visual/link1.dae
- link panda_link2: mass 2.0 -> 2.36; geometry collision mesh filename=package://franka_description/meshes/collision/link2.stl; visual mesh filename=package://franka_description/meshes/visual/link2.dae
- link panda_link3: mass 2.0 -> 2.38; geometry collision mesh filename=package://franka_description/meshes/collision/link3.stl; visual mesh filename=package://franka_description/meshes/visual/link3.dae
- link panda_link4: mass 2.0 -> 2.43; geometry collision mesh filename=package://franka_description/meshes/collision/link4.stl; visual mesh filename=package://franka_description/meshes/visual/link4.dae
- link panda_link5: mass 2.0 -> 3.5; geometry collision mesh filename=package://franka_description/meshes/collision/link5.stl; visual mesh filename=package://franka_description/meshes/visual/link5.dae
- link panda_link6: mass 1.0 -> 1.47; geometry collision mesh filename=package://franka_description/meshes/collision/link6.stl; visual mesh filename=package://franka_description/meshes/visual/link6.dae
- link panda_link7: mass 0.2 -> 0.45; geometry collision mesh filename=package://franka_description/meshes/collision/link7.stl; visual mesh filename=package://franka_description/meshes/visual/link7.dae
- link panda_link8: mass None -> 1e-10
Joints:
- removed joint eef_to_box
- removed joint panda_joint_world
- added joint panda_finger_joint1: type prismatic, parent panda_hand, child panda_leftfinger, origin xyz=0 0 0.0584 rpy=0 0 0, axis 0 1 0, limit lower=0.0 upper=0.04 effort=20 velocity=0.2
- added joint panda_finger_joint2: type prismatic, parent panda_hand, child panda_rightfinger, origin xyz=0 0 0.0584 rpy=0 0 0, axis 0 -1 0, limit lower=0.0 upper=0.04 effort=20 velocity=0.2, mimic joint=panda_finger_joint1
- added joint panda_hand_joint: type fixed, parent panda_link8, child panda_hand, origin xyz=0 0 0 rpy=0 0 -0.785398163397
- joint panda_joint1: limit lower=-2.9671 upper=2.9671 effort=87 velocity=2.5 -> lower=-2.8973 upper=2.8973 effort=87 velocity=2.1750
- joint panda_joint2: limit lower=-1.8326 upper=1.8326 effort=87 velocity=2.5 -> lower=-1.7628 upper=1.7628 effort=87 velocity=2.1750; origin xyz=0 0 0 rpy=-1.570796326794897 0 0 -> xyz=0 0 0 rpy=-1.57079632679 0 0
- joint panda_joint3: limit lower=-2.9671 upper=2.9671 effort=87 velocity=2.5 -> lower=-2.8973 upper=2.8973 effort=87 velocity=2.1750; origin xyz=0 -0.316 0 rpy=1.570796326794897 0 0 -> xyz=0 -0.316 0 rpy=1.57079632679 0 0
- joint panda_joint4: limit lower=-3.1416 upper=0.0873 effort=87 velocity=2.5 -> lower=-3.0718 upper=-0.0698 effort=87 velocity=2.1750; origin xyz=0.0825 0 0 rpy=1.570796326794897 0 0 -> xyz=0.0825 0 0 rpy=1.57079632679 0 0
- joint panda_joint5: limit lower=-2.9671 upper=2.9671 effort=12 velocity=3 -> lower=-2.8973 upper=2.8973 effort=12 velocity=2.6100; origin xyz=-0.0825 0.384 0 rpy=-1.570796326794897 0 0 -> xyz=-0.0825 0.384 0 rpy=-1.57079632679 0 0
- joint panda_joint6: limit lower=-0.0873 upper=3.8223 effort=12 velocity=3 -> lower=-0.0175 upper=3.7525 effort=12 velocity=2.6100; origin xyz=0 0 0 rpy=1.570796326794897 0 0 -> xyz=0 0 0 rpy=1.57079632679 0 0
- joint panda_joint7: limit lower=-2.9671 upper=2.9671 effort=12 velocity=3 -> lower=-2.8973 upper=2.8973 effort=12 velocity=2.6100; origin xyz=0.088 0 0 rpy=1.570796326794897 0 0 -> xyz=0.088 0 0 rpy=1.57079632679 0 0
- joint panda_joint8: axis (none) -> 0 0 0

Commit message: [robots]: Add EE frame in Franka

File: robots/franka/franka.urdf (robot description, URDF)
Before this commit: robot panda, 12 links, 11 joints
Links:
- added link panda_ee, mass 1e-10
Joints:
- added joint panda_ee_joint: type fixed, parent panda_link8, child panda_ee, origin xyz=0 0 0.103 rpy=0 0 -0.785398163397
