Commit message: [tiago]: add differential drive

File: utheque/tiago/tiago_steel.urdf (robot description, URDF)
Before this commit: robot tiago, 55 links, 54 joints
Joints:
- joint caster_back_left_1_joint: type fixed -> continuous
- joint caster_back_left_2_joint: type fixed -> continuous
- joint caster_back_right_1_joint: type fixed -> continuous
- joint caster_back_right_2_joint: type fixed -> continuous
- joint caster_front_left_1_joint: type fixed -> continuous
- joint caster_front_left_2_joint: type fixed -> continuous
- joint caster_front_right_1_joint: type fixed -> continuous
- joint caster_front_right_2_joint: type fixed -> continuous
- joint wheel_left_joint: limit lower=-1.7976931348623157e+308 upper=1.7976931348623157e+308 effort=6.0 velocity=10.152284264 -> effort=6.0 velocity=10.152284264; type revolute -> continuous
- joint wheel_right_joint: limit lower=-1.7976931348623157e+308 upper=1.7976931348623157e+308 effort=6.0 velocity=10.152284264 -> effort=6.0 velocity=10.152284264; type revolute -> continuous

Commit message: Fix Tiago URDF [ci skip]

File: utheque/tiago/tiago_steel.urdf (robot description, URDF)
Before this commit: robot tiago, 55 links, 54 joints
Joints:
- joint gripper_right_finger_joint: limit lower=0.002 upper=0.034 effort=16 velocity=0.4 -> lower=0.002 upper=0.034 effort=50 velocity=0.4; type fixed -> prismatic
