Commit message: Better collisions for gripper of Vx300

File: utheque/vx300/vx300.urdf (robot description, URDF)
Before this commit: robot vx300, 13 links, 12 joints
Links:
- link vx300/left_finger_link: geometry collision box size=0.08 0.02575 0.05; visual mesh filename=package://interbotix_xsarm_descriptions/vx300_meshes/vx300_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 scale=0.001 0.001 0.001
- link vx300/right_finger_link: geometry collision box size=0.08 0.02575 0.05; visual mesh filename=package://interbotix_xsarm_descriptions/vx300_meshes/vx300_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 scale=0.001 0.001 0.001

Commit message: Update Vx300 URDF [ci skip]

File: utheque/vx300/vx300.urdf (robot description, URDF)
Before this commit: robot vx300, 13 links, 12 joints
Links:
- link vx300/gripper_bar_link: geometry visual mesh filename=package://interbotix_xsarm_descriptions/vx300_meshes/vx300_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 scale=0.001 0.001 0.001
- link vx300/left_finger_link: geometry collision box size=0.07 0.02575 0.05; visual mesh filename=package://interbotix_xsarm_descriptions/vx300_meshes/vx300_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 scale=0.001 0.001 0.001
- link vx300/right_finger_link: geometry collision box size=0.07 0.02575 0.05; visual mesh filename=package://interbotix_xsarm_descriptions/vx300_meshes/vx300_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 scale=0.001 0.001 0.001
